File: design_files/ASD2205.brd (EAGLE design)
At the start: 25.8 x 25 mm, 12 parts, among them J1 SM02B-SRSS, J2 DF12-32-DS, J7 DM3D-SF, U1 TSOP57438, U2 TS922IDT

Commit message: Update hardware rev
Parts:
- removed J7: DM3D-SF, tinycircuits:SD_CARD
- added C5: 0.1uF, tinycircuits:C0402
- added J3: DF12-32-DS, tinycircuits:DF12-32-DS
- added R2: 100K, tinycircuits:0402
- C2: value 0.1uF -> 10uF; device tinycircuits:C0402 -> tinycircuits:C0603
- C3: value 100uF -> 0.1uF; device tinycircuits:C1206 -> tinycircuits:C0402
- C4: value 10nF -> 0.1uF
- C6: value 10uF -> 0.1uF; device tinycircuits:C0603 -> tinycircuits:C0402
- J1: value SM02B-SRSS -> DM3D-SF; device tinycircuits:JST_SH_2X1 -> tinycircuits:SD_CARD
- J2: value DF12-32-DS -> SM02B-SRSS; device tinycircuits:DF12-32-DS -> tinycircuits:JST_SH_2X1
- R1: value 1.00K -> 100K
- U1: value TSOP57438 -> NCP2820; device tinycircuits:TSOP57 -> tinycircuits:WSON-8
- U2: value TS922IDT -> TSOP57438; device tinycircuits:SO-08-COMPACT -> tinycircuits:TSOP57
- moved C6 16.4 mm to (25.0, 10.1), turned to 0 degrees
- moved U1 14.4 mm to (16.5, 19.0), turned to 0 degrees
- moved U2 13.4 mm to (25.0, 7.40), turned to 180 degrees
- moved J2 10.9 mm to (21.0, 24.4), turned to 180 degrees
- moved C2 10.7 mm to (22.9, 20.6), turned to 270 degrees
- moved J1 10.4 mm to (30.5, 28.6)
- moved C1 8.42 mm to (13.7, 20.1), turned to 90 degrees
- moved C3 6.32 mm to (14.9, 18.7), turned to 90 degrees
- moved R1 2.61 mm to (18.2, 18.7), turned to 270 degrees
- moved C4 1.79 mm to (18.8, 20.3), turned to 180 degrees
Connections:
- removed net N$1: C3.1, U2.6, U2.7
- removed net N$2: C3.2, J1.2
- removed net N$7: C4.1, R1.2, U2.5
- removed net N$9: R1.1, U2.1, U2.2
- new net N$11: C4.2, R1.1
- new net N$12: C5.2, R2.1
- new net N$3: R1.2, U1.4
- new net N$4: R2.2, U1.3
- new net SPK+: J2.2, U1.5
- new net SPK-: J2.1, U1.8
- net +3V3: now also J3.6; no longer J2.6
- net +5V: now also J3.8; no longer J2.8
- net AD0: now also C4.1, J3.11; no longer J2.11, U2.3
- net AD1: now also J3.9; no longer J2.9
- net AD2: now also J3.7; no longer J2.7
- net AD3: now also J3.5; no longer J2.5
- net AD4/SDA: now also J3.3; no longer J2.3
- net AD5/SCL: now also J3.1; no longer J2.1
- net AREF: now also J3.13; no longer J2.13
- net GND: now also C3.2, C5.1, J1.6, J3.12, J3.14, U1.7, U1.9, U2.6, U2.8; no longer C4.2, J1.1, J2.12, J2.14, J7.6, U1.6, U1.8, U2.4
- net IO0: now also J3.24; no longer J2.24
- net IO1: now also J3.26; no longer J2.26
- net IO2: now also J3.28; no longer J2.28
- net IO3: now also J3.30, U2.1; no longer J2.30, U1.1
- net IO4: now also J3.32; no longer J2.32
- net IO5: now also J3.31; no longer J2.31
- net IO6: now also J3.29; no longer J2.29
- net IO7: now also J3.27; no longer J2.27
- net IO8: now also J3.25; no longer J2.25
- net IO9: now also J3.23; no longer J2.23
- net MISO: now also J1.7, J3.17; no longer J2.17, J7.7
- net MOSI: now also J1.3, J3.19; no longer J2.19, J7.3
- net RESET: now also J3.22; no longer J2.22
- net RSV0: now also J3.20; no longer J2.20
- net RSV1: now also J3.18; no longer J2.18
- net RSV2: now also J3.16; no longer J2.16
- net SCK: now also J1.5, J3.15; no longer J2.15, J7.5
- net SS: now also J1.2, J3.21; no longer J2.21, J7.2
- net VBATT: now also J3.4; no longer J2.4
- net VCC: now also C3.1, J1.4, J3.2, U1.1, U1.2, U1.6, U2.5; no longer J2.2, J7.4, U1.5, U2.8
- net VIN: now also J3.10; no longer J2.10
Routing:
- net SPK-: track 0.00 -> 8.75 mm
- net N$1: track 7.49 -> 0.00 mm
- net N$9: track 6.58 -> 0.00 mm
- net AD0: track 13.2 -> 7.48 mm, vias 2 -> 0
- net VCC: track 42.7 -> 47.6 mm, vias 4 -> 5
- net SPK+: track 0.00 -> 4.75 mm
- net N$4: track 0.00 -> 3.68 mm
- net N$2: track 3.60 -> 0.00 mm
- net N$7: track 2.92 -> 0.00 mm
- net GND: track 3.37 -> 6.09 mm, vias 14 -> 22
- net N$12: track 0.00 -> 1.10 mm
- net N$11: track 0.00 -> 1.05 mm
- net N$3: track 0.00 -> 0.96 mm
Other:
- board text added: "3"
- board text added: "ASD2205 - Rev3"
- board text removed: "2"
- board text removed: "ASD2205 - Rev2"
