File: design_files/ASD2205.sch (EAGLE design)
At the start: 11 parts, among them J1 SM02B-SRSS, J2 DF12-32-DS, J7 DM3D-SF, U1 TSOP57438, U2 TS922IDT

Commit message: Update hardware rev
Parts:
- removed J7: DM3D-SF, tinycircuits:AS-ITM-00047
- added C5: 0.1uF, tinycircuits:AS-ITM-00008
- added J3: DF12-32-DS, tinycircuits:AS-ITM-00012
- added R2: 100K, tinycircuits:AS-ITM-00004
- C1: PARTNO AS-ITM-00002 -> (none); VALUE 10uF -> (none)
- C2: value 0.1uF -> 10uF; device tinycircuits:AS-ITM-00008 -> tinycircuits:AS-ITM-00002; PARTNO (none) -> AS-ITM-00002; VALUE (none) -> 10uF
- C3: value 100uF -> 0.1uF; device tinycircuits:AS-ITM-00095 -> tinycircuits:AS-ITM-00008
- C4: value 10nF -> 0.1uF; device tinycircuits:AS-ITM-00084 -> tinycircuits:AS-ITM-00008
- C6: value 10uF -> 0.1uF; device tinycircuits:AS-ITM-00002 -> tinycircuits:AS-ITM-00008
- J1: value SM02B-SRSS -> DM3D-SF; device tinycircuits:AS-ITM-00231 -> tinycircuits:AS-ITM-00047
- J2: value DF12-32-DS -> SM02B-SRSS; device tinycircuits:AS-ITM-00012 -> tinycircuits:AS-ITM-00231; PARTNO AS-ITM-00012 -> (none); VALUE DF12-32-DS -> (none)
- R1: value 1.00K -> 100K; device tinycircuits:AS-ITM-00003 -> tinycircuits:AS-ITM-00004; PARTNO AS-ITM-00003 -> (none); VALUE 1.00K -> (none)
- U1: value TSOP57438 -> NCP2820; device tinycircuits:AS-ITM-00360 -> tinycircuits:AS-ITM-00370
- U2: value TS922IDT -> TSOP57438; device tinycircuits:AS-ITM-000922 -> tinycircuits:AS-ITM-00360
Connections:
- removed net N$1: C3.1, U2.2IN-, U2.2OUT
- removed net N$2: C3.2, J1.1
- removed net N$7: C4.1, R1.2, U2.2IN+
- removed net N$9: R1.1, U2.IN1-, U2.OUT1
- new net N$11: C4.2, R1.1
- new net N$12: C5.2, R2.1
- new net N$3: R1.2, U1.IN-
- new net N$4: R2.2, U1.IN+
- new net SPK+: J2.1, U1.OUT+
- new net SPK-: J2.2, U1.OUT-
- net +3V3: now also J3.6; no longer J2.6
- net +5V: now also J3.8; no longer J2.8
- net AD0: now also C4.1, J3.11; no longer J2.11, U2.IN1+
- net AD1: now also J3.9; no longer J2.9
- net AD2: now also J3.7; no longer J2.7
- net AD3: now also J3.5; no longer J2.5
- net AD4/SDA: now also J3.3; no longer J2.3
- net AD5/SCL: now also J3.1; no longer J2.1
- net AREF: now also J3.13; no longer J2.13
- net GND: now also C3.2, C5.1, J1.VSS, J3.12, J3.14, U2.GND; no longer C4.2, J1.2, J2.12, J2.14, J7.VSS, U2.VCC-
- net IO0: now also J3.24; no longer J2.24
- net IO1: now also J3.26; no longer J2.26
- net IO2: now also J3.28; no longer J2.28
- net IO3: now also J3.30, U2.OUT; no longer J2.30, U1.OUT
- net IO4: now also J3.32; no longer J2.32
- net IO5: now also J3.31; no longer J2.31
- net IO6: now also J3.29; no longer J2.29
- net IO7: now also J3.27; no longer J2.27
- net IO8: now also J3.25; no longer J2.25
- net IO9: now also J3.23; no longer J2.23
- net MISO: now also J1.DAT0, J3.17; no longer J2.17, J7.DAT0
- net MOSI: now also J1.CMD, J3.19; no longer J2.19, J7.CMD
- net RESET: now also J3.22; no longer J2.22
- net RSV0: now also J3.20; no longer J2.20
- net RSV1: now also J3.18; no longer J2.18
- net RSV2: now also J3.16; no longer J2.16
- net SCK: now also J1.CLK, J3.15; no longer J2.15, J7.CLK
- net SS: now also J1.CD/DAT3, J3.21; no longer J2.21, J7.CD/DAT3
- net VBATT: now also J3.4; no longer J2.4
- net VCC: now also C3.1, J1.VDD, J3.2, U1.!SDN, U1.VCC, U2.VIN; no longer J2.2, J7.VDD, U1.VIN, U2.VCC+
- net VIN: now also J3.10; no longer J2.10
Other:
- note added: "3"
- note added: "Hand Populated: -"
- note removed: "2"
- note removed: "Hand Populated: U1"
- moved on the sheet: C1, C2, C3, C4, C6, R1
